File: Left/Switch.kicad_sch (KiCad schematic)
At the start: 4 parts, among them Q2 AO3407, U2 Button, U3 MAX16054

Commit message: Finished left hand
Connections:
- no-connect marks 2 -> 3
Changed lines of the file:
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@@
   (junction (at 121.285 114.3) (diameter 0) (color 0 0 0 0)
   )
+  (no_connect (at 98.425 113.03))
   (no_connect (at 119.38 105.41))
   (no_connect (at 98.425 105.41))
@@
   )
   (symbol (lib_id "Library:Button") (at 100.33 111.125 180) (unit 1)
-    (in_bom yes) (on_board yes) (fields_autoplaced)
-    (property "Reference" "U2" (id 0) (at 98.425 113.03 0))
-    (property "Value" "Button" (id 1) (at 98.425 115.57 0))
+    (in_bom yes) (on_board yes)
+    (property "Reference" "U2" (id 0) (at 98.425 114.935 0))
+    (property "Value" "Button" (id 1) (at 98.425 116.205 0))
     (property "Footprint" "Library:Button" (id 2) (at 98.425 104.775 0)
       (effects (font (size 1.27 1.27)) hide)
@@
     (pin "2")
     (pin "3")
+    (pin "4")
   )
   (symbol (lib_id "Library:MAX16054") (at 111.125 110.49 0) (unit 1)
